File: HaRTK/HaRTK.kicad_pcb (KiCad board)
At the start: 4 copper layers, 65 x 40 mm, 22 parts, among them P1 Telem RF, P2 GPS RF, P3 PPS, P4 CONN_01X06, P5 Bat holder, U1 RaspberryPi, U2 LM1117, U3 RFM22B, U4 NV08C-CSM

Commit message: First revision
Parts:
- removed C3: 1uF, Capacitors_SMD:C_0805_HandSoldering
- removed C4: 22pF, Capacitors_SMD:C_0805_HandSoldering
- added G***: LOGO, logo:LOGO, F.Cu at (117.5, 79.6)
- GPS Com: renamed from D4
- RPi Com: renamed from D3
- moved Link 40.0 mm to (122.5, 95.0)
- moved PPS 40.0 mm to (162.5, 95.0)
- moved C1 14.1 mm to (118.0, 70.0), turned to 180 degrees
- moved P5 5.46 mm to (130.9, 75.6)
- moved U2 3.40 mm to (116.8, 76.5), turned to 270 degrees
- moved C2 1.76 mm to (125.0, 77.5), turned to 270 degrees
- moved U4 0.51 mm to (153.4, 78.5), turned to 180 degrees
- moved RP1 0.50 mm to (152.5, 95.0)
- renumbered D1 to 3.3V, D2 to Amp, D8 to Error, P2 to GPS, D6 to Link, P1 to Link, D5 to Lock, P3 to PPS, D7 to RTK
Connections:
- U2 pad 1: (no net) -> +5V
- U2 pad 2: (no net) -> GND
- U2 pad 3: (no net) -> +3V3
Routing:
- net GND: track 0.00 -> 130.9 mm, vias 0 -> 101
- net /TX_BINR_NVC: track 0.00 -> 72.8 mm, vias 0 -> 2
- net /SDA: track 0.00 -> 71.0 mm
- net /SCL: track 0.00 -> 64.0 mm
- net /ANTFLAG_NVC: track 0.00 -> 63.7 mm, vias 0 -> 3
- net /SCK_RFM22B: track 0.00 -> 53.7 mm, vias 0 -> 1
- net /RX_BINR_NVC: track 0.00 -> 51.1 mm
- net /RTK_SOLUTION: track 0.00 -> 49.9 mm, vias 0 -> 1
- net Net-(D6-Pad1): track 0.00 -> 49.6 mm, vias 0 -> 3
- net /GPS_LOCK: track 0.00 -> 48.2 mm, vias 0 -> 1
- net /ERROR: track 0.00 -> 45.2 mm, vias 0 -> 1
- net Net-(D8-Pad1): track 0.00 -> 43.5 mm, vias 0 -> 1
- net /BASE_DETECTED: track 0.00 -> 38.7 mm, vias 0 -> 1
- net /SLEEPFLAG_NVC: track 0.00 -> 37.9 mm, vias 0 -> 1
- net /GPIO1_RFM22B: track 0.00 -> 37.3 mm, vias 0 -> 2
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- added copper zone on In2.Cu, net +3V3
- added copper zone on B.Cu, net GND
- added copper zone on F.Cu, net GND
- added copper zone on In1.Cu, net GND
- added copper zone on In2.Cu, net GND
Other:
- rule trace_min: 0.2 -> 0.127
- rule via_min_drill: 0.3 -> 0.254
- rule via_min_size: 0.4 -> 0.454
- board text added: "H. Pienaar June 2016 Rev. 1"
- board text added: "RTK RPi GPS"
